File: bootcamp-elec.kicad_pcb (KiCad board)
At the start: 2 copper layers, 0 parts

Commit message: pcb design done
Parts:
- added C1: 12pF, bootcamp-elec:C_0805_2012Metric, F.Cu at (208.7, 116.2)
- added C2: 12pF, bootcamp-elec:C_0805_2012Metric, F.Cu at (209.2, 108.9)
- added C3: 100nF, bootcamp-elec:C_0805_2012Metric, F.Cu at (220.9, 123.8)
- added C4: 100nF, bootcamp-elec:C_0805_2012Metric, F.Cu at (222.6, 136.3)
- added C6: 1uF, bootcamp-elec:C_0805_2012Metric, F.Cu at (223.0, 107.5)
- added C7: 100nF, bootcamp-elec:C_0805_2012Metric, F.Cu at (223.0, 111.2)
- added D1: Green, bootcamp-elec:LED_0805_2012Metric, F.Cu at (215.0, 127.2)
- added D2: Red, bootcamp-elec:LED_0805_2012Metric, F.Cu at (221.0, 111.2)
- added G***: LOGO, bootcamp-elec:arrows-silkscreen, F.Cu at (228.3, 104.0)
- added G***: LOGO, bootcamp-elec:flags-silkscreen, F.Cu at (203.6, 103.9)
- added J1: ~, bootcamp-elec:PinHeader_1x12_P2.54mm_Vertical, F.Cu at (203.6, 136.5)
- added J2: ~, bootcamp-elec:PinHeader_1x12_P2.54mm_Vertical, F.Cu at (228.4, 108.5)
- added J3: FTDI, bootcamp-elec:PinHeader_1x06_P2.54mm_Vertical, F.Cu at (209.6, 104.0)
- added R1: 330, bootcamp-elec:R_0805_2012Metric, F.Cu at (217.1, 127.2)
- added R2: 10K, bootcamp-elec:R_0805_2012Metric, F.Cu at (221.0, 107.5)
- added R3: 10K, bootcamp-elec:R_0805_2012Metric, F.Cu at (209.3, 136.3)
- added SW1: SW_Push, bootcamp-elec:SW_Tact_6X6mm_H5mm_SMD, F.Cu at (216.0, 134.7)
- added U1: ATmega328P-A, bootcamp-elec:TQFP-32_7x7mm_P0.8mm, F.Cu at (216.0, 118.3)
- added Y1: 16MHz, bootcamp-elec:Crystal_SMD_3225-4Pin_3.2x2.5mm, F.Cu at (208.3, 112.5)
Routing:
- net DTR: track 0.00 -> 83.9 mm, vias 0 -> 1
- net RAW: track 0.00 -> 80.9 mm, vias 0 -> 3
- net D10: track 0.00 -> 39.4 mm
- net RXI: track 0.00 -> 27.5 mm
- net MOSI: track 0.00 -> 26.6 mm
- net TXO: track 0.00 -> 24.0 mm, vias 0 -> 1
- net MISO: track 0.00 -> 23.3 mm
- net D9: track 0.00 -> 18.4 mm
- net D4: track 0.00 -> 17.0 mm, vias 0 -> 1
- net D2: track 0.00 -> 16.8 mm, vias 0 -> 1
- net D8: track 0.00 -> 16.3 mm
- net D3: track 0.00 -> 15.4 mm, vias 0 -> 1
- net SCK: track 0.00 -> 14.9 mm
- net D7: track 0.00 -> 14.2 mm
- net D6: track 0.00 -> 12.6 mm
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- added copper zone on B.Cu, net GND
- added copper zone on F.Cu, net GND
Other:
- board outline added: 28.9 x 36.4 mm
